Commit message: [lucifer][add]: nav2 navigation package and configs

File: src/tianbot_description_ros2/urdf/tianracer_base.xacro (robot description, xacro)
@@ -20,4 +20,28 @@
     </link>
     <link name="base_link">
+        <inertial>
+            <origin xyz="0 0 ${chassis_height/2}" rpy="0 0 0" />
+            <mass value="${body_mass}" />
+            <inertia ixx="${body_mass/12 * (chassis_width*chassis_width + chassis_height*chassis_height)}"
+                ixy="0" ixz="0"
+                iyy="${body_mass/12 * (chassis_length*chassis_length + chassis_height*chassis_height)}"
+                iyz="0"
+                izz="${body_mass/12 * (chassis_length*chassis_length + chassis_width*chassis_width)}" />
+        </inertial>
+        <visual>
+            <origin xyz="0 0 ${chassis_height/2}" rpy="0 0 0" />
+            <geometry>
+                <box size="${chassis_length} ${chassis_width} ${chassis_height}" />
+            </geometry>
+            <material name="black">
+                <color rgba="0.15 0.15 0.15 1.0" />
+            </material>
+        </visual>
+        <collision>
+            <origin xyz="0 0 ${chassis_height/2}" rpy="0 0 0" />
+            <geometry>
+                <box size="${chassis_length} ${chassis_width} ${chassis_height}" />
+            </geometry>
+        </collision>
     </link>
     <joint name="base_joint" type="fixed">
@@ -26,36 +50,4 @@
         <origin xyz="0.0 0.0 ${wheel_radius}" rpy="0 0 0" />
     </joint>
-    <!-- CHASSIS -->
-    <link name="chassis_link">
-        <inertial>
-            <origin xyz="0 0 ${chassis_height/2}" rpy="0 0 0" />
-            <mass value="${body_mass}" />
-            <inertia ixx="${body_mass/12 * (chassis_width*chassis_width + chassis_height*chassis_height)}"
-                ixy="0" ixz="0"
-                iyy="${body_mass/12 * (chassis_length*chassis_length + chassis_height*chassis_height)}"
-                iyz="0"
-                izz="${body_mass/12 * (chassis_length*chassis_length + chassis_width*chassis_width)}" />
-        </inertial>
-        <visual>
-            <origin xyz="0 0 ${chassis_height/2}" rpy="0 0 0" />
-            <geometry>
-                <box size="${chassis_length} ${chassis_width} ${chassis_height}" />
-            </geometry>
-            <material name="black">
-                <color rgba="0.15 0.15 0.15 1.0" />
-            </material>
-        </visual>
-        <collision>
-            <origin xyz="0 0 ${chassis_height/2}" rpy="0 0 0" />
-            <geometry>
-                <box size="${chassis_length} ${chassis_width} ${chassis_height}" />
-            </geometry>
-        </collision>
-    </link>
-    <joint name="chassis_joint" type="fixed">
-        <parent link="base_link" />
-        <child link="chassis_link" />
-        <origin xyz="0.0 0.0 0.0" rpy="0 0 0" />
-    </joint>
     <!-- FRONT LEFT WHEEL -->
     <link name="fr_left_steer_link">
@@ -72,5 +64,5 @@
     <joint name="fr_left_steer_joint" type="revolute">
         <origin xyz="${front_wheel_x} ${wheel_y} ${wheel_radius}" rpy="0 0 0" />
-        <parent link="chassis_link" />
+        <parent link="base_link" />
         <child link="fr_left_steer_link" />
         <axis xyz="0 0 1" />
@@ -125,5 +117,5 @@
     <joint name="fr_right_steer_joint" type="revolute">
         <origin xyz="${front_wheel_x} ${-wheel_y} ${wheel_radius}" rpy="0 0 0" />
-        <parent link="chassis_link" />
+        <parent link="base_link" />
         <child link="fr_right_steer_link" />
         <axis xyz="0 0 1" />
@@ -193,5 +185,5 @@
     <joint name="re_left_wheel_joint" type="continuous">
         <origin xyz="${rear_wheel_x} ${wheel_y} ${wheel_radius}" rpy="0 0 0" />
-        <parent link="chassis_link" />
+        <parent link="base_link" />
         <child link="re_left_wheel_link" />
         <axis xyz="0 1 0" />
@@ -228,5 +220,5 @@
     <joint name="re_right_wheel_joint" type="continuous">
         <origin xyz="${rear_wheel_x} ${-wheel_y} ${wheel_radius}" rpy="0 0 0" />
-        <parent link="chassis_link" />
+        <parent link="base_link" />
         <child link="re_right_wheel_link" />
         <axis xyz="0 1 0" />
@@ -258,10 +250,10 @@
     </link>
     <joint name="camera_joint" type="fixed">
-        <parent link="chassis_link"/>
+        <parent link="base_link"/>
         <child link="camera_link"/>
         <origin rpy="0 0 0" xyz="${front_wheel_x} 0 ${chassis_height}"/>
     </joint>
-    <!-- LIDAR: 摄像头往后3cm -->
-    <link name="lidar_link">
+    <!-- LASER: 摄像头往后3cm -->
+    <link name="laser_link">
         <visual>
             <geometry>
@@ -285,7 +277,7 @@
         </inertial>
     </link>
-    <joint name="lidar_joint" type="fixed">
-        <parent link="chassis_link"/>
-        <child link="lidar_link"/>
+    <joint name="laser_joint" type="fixed">
+        <parent link="base_link"/>
+        <child link="laser_link"/>
         <origin rpy="0 0 0" xyz="${front_wheel_x - 0.03} 0 ${chassis_height}"/>
     </joint>
@@ -314,5 +306,5 @@
     </link>
     <joint name="imu_joint" type="fixed">
-        <parent link="chassis_link"/>
+        <parent link="base_link"/>
         <child link="imu_link"/>
         <origin rpy="0 0 0" xyz="0 0 ${chassis_height/2}"/>

File: src/tianbot_description_ros2/urdf/tianracer_gazebo_core.xacro (robot description, xacro)
@@ -4,5 +4,5 @@
     <!-- Gazebo is unable to use the same <material> tags that are already in the URDF (that RViz uses). -->
     <!-- Instead, we need to add gazebo tags for our links that refer to Gazebo materials -->
-    <gazebo reference="chassis_link">
+    <gazebo reference="base_link">
         <material>Gazebo/White</material>
         <mu1>0.5</mu1>
@@ -70,12 +70,12 @@
         </sensor>
     </gazebo>
-    <!-- LIDAR -->
-    <gazebo reference="lidar_link">
+    <!-- LASER -->
+    <gazebo reference="laser_link">
         <material>Gazebo/Black</material>
         <mu1>1.0</mu1>
         <mu2>1.0</mu2>
     </gazebo>
-    <gazebo reference="lidar_link">
-        <sensor name="lidar_sensor" type="gpu_ray">
+    <gazebo reference="laser_link">
+        <sensor name="laser_sensor" type="gpu_ray">
             <always_on>true</always_on>
             <visualize>true</visualize>
@@ -102,10 +102,10 @@
                 </noise>
             </ray>
-            <plugin name="lidarscan" filename="libgazebo_ros_ray_sensor.so">
+            <plugin name="laserscan" filename="libgazebo_ros_ray_sensor.so">
                 <ros>
                     <remapping>~/out:=scan</remapping>
                 </ros>
                 <output_type>sensor_msgs/LaserScan</output_type>
-                <frame_name>lidar_link</frame_name>
+                <frame_name>laser_link</frame_name>
             </plugin>
         </sensor>
@@ -279,5 +279,5 @@
     <joint name="virtual_steering_wheel_joint" type="revolute">
         <origin xyz="-0.32 0.0 0.0" rpy="0.0 0.0 0.0" />
-        <parent link="chassis_link" />
+        <parent link="base_link" />
         <child link="virtual_steer_link" />
         <axis xyz="-1 0 0" />

Commit message: [lucifer][update]: how to use gpu in nav2

File: src/tianbot_description_ros2/urdf/tianracer_base.xacro (robot description, xacro)
@@ -67,5 +67,6 @@
         <child link="fr_left_steer_link" />
         <axis xyz="0 0 1" />
-        <limit upper="0.6" lower="-0.6" effort="-1.0" velocity="-1.0" />
+        <limit upper="0.6" lower="-0.6" effort="100" velocity="10" />
+        <dynamics damping="10.0" friction="1.0" />
     </joint>
     <link name="fr_left_wheel_link">
@@ -120,5 +121,6 @@
         <child link="fr_right_steer_link" />
         <axis xyz="0 0 1" />
-        <limit upper="0.6" lower="-0.6" effort="-1.0" velocity="-1.0" />
+        <limit upper="0.6" lower="-0.6" effort="100" velocity="10" />
+        <dynamics damping="10.0" friction="1.0" />
     </joint>
     <link name="fr_right_wheel_link">
