Commit message: [lucifer][update]: run success, just save

File: src/tianbot_description_ros2/urdf/tianbot_ackermann.urdf.xacro (robot description, xacro)
@@ -7,4 +7,6 @@
   <xacro:property name="wheel_radius" value="0.065"/>
   <xacro:property name="wheel_width" value="0.04"/>
+  <xacro:property name="wheel_mass" value="3.0"/>
+  <xacro:property name="steering_mass" value="0.01"/>
   <!-- 轮子位置：前轮距前端6cm，后轮距后端4cm -->
   <xacro:property name="front_wheel_x" value="${chassis_length/2 - 0.06}"/>
@@ -16,4 +18,6 @@
   <!-- Base Footprint -->
   <link name="base_footprint"/>
+  <!-- Base Link -->
+  <link name="base_link"/>
   <joint name="base_footprint_joint" type="fixed">
     <parent link="base_footprint"/>
@@ -21,6 +25,6 @@
     <origin xyz="0 0 ${wheel_radius}" rpy="0 0 0"/>
   </joint>
-  <!-- Base Link -->
-  <link name="base_link">
+  <!-- Chassis Link -->
+  <link name="chassis_link">
     <visual>
       <origin xyz="0 0 ${chassis_height/2}" rpy="0 0 0"/>
@@ -44,18 +48,28 @@
     </inertial>
   </link>
+  <joint name="chassis_joint" type="fixed">
+    <parent link="base_link"/>
+    <child link="chassis_link"/>
+    <origin xyz="0 0 0" rpy="0 0 0"/>
+  </joint>
   <!-- 前轮转向宏 -->
   <xacro:macro name="front_wheel" params="prefix reflect">
     <joint name="${prefix}_steer_joint" type="revolute">
-      <parent link="base_link"/>
+      <parent link="chassis_link"/>
       <child link="${prefix}_steer_link"/>
-      <origin xyz="${front_wheel_x} ${reflect*wheel_y} 0" rpy="0 0 0"/>
+      <origin xyz="${front_wheel_x} ${reflect*wheel_y} ${wheel_radius}" rpy="0 0 0"/>
       <axis xyz="0 0 1"/>
-      <limit lower="-0.5" upper="0.5" effort="100" velocity="2.0"/>
+      <!-- <limit lower="-0.6" upper="0.6" effort="-1.0" velocity="-1.0"/> -->
+      <limit lower="-0.6" upper="0.6" effort="100" velocity="-1.0"/>
     </joint>
     <link name="${prefix}_steer_link">
       <inertial>
-        <mass value="0.1"/>
+        <mass value="${steering_mass}"/>
         <origin xyz="0 0 0" rpy="0 0 0"/>
-        <inertia ixx="0.001" ixy="0" ixz="0" iyy="0.001" iyz="0" izz="0.001"/>
+        <inertia ixx="${steering_mass/12*(3*wheel_radius*wheel_radius + wheel_width*wheel_width)}"
+                 ixy="0" ixz="0"
+                 iyy="${steering_mass/12*(3*wheel_radius*wheel_radius + wheel_width*wheel_width)}"
+                 iyz="0"
+                 izz="${steering_mass/2 * wheel_radius*wheel_radius}"/>
       </inertial>
     </link>
@@ -65,4 +79,6 @@
       <origin xyz="0 0 0" rpy="0 0 0"/>
       <axis xyz="0 1 0"/>
+      <dynamics damping="0.5" friction="0.8"/>
+      <!-- <limit lower="-3.14159" upper="3.14159" effort="200" velocity="-1"/> -->
     </joint>
     <link name="${prefix}_wheel">
@@ -83,7 +99,11 @@
       </collision>
       <inertial>
-        <mass value="1.0"/>
+        <mass value="${wheel_mass}"/>
         <origin xyz="0 0 0" rpy="0 0 0"/>
-        <inertia ixx="0.005" ixy="0" ixz="0" iyy="0.005" iyz="0" izz="0.005"/>
+        <inertia ixx="${wheel_mass/12*(3*wheel_radius*wheel_radius + wheel_width*wheel_width)}"
+                 ixy="0" ixz="0"
+                 iyy="${wheel_mass/12*(3*wheel_radius*wheel_radius + wheel_width*wheel_width)}"
+                 iyz="0"
+                 izz="${wheel_mass/2 * wheel_radius*wheel_radius}"/>
       </inertial>
     </link>
@@ -92,8 +112,10 @@
   <xacro:macro name="rear_wheel" params="prefix reflect">
     <joint name="${prefix}_wheel_joint" type="continuous">
-      <parent link="base_link"/>
+      <parent link="chassis_link"/>
       <child link="${prefix}_wheel"/>
-      <origin xyz="${rear_wheel_x} ${reflect*wheel_y} 0" rpy="0 0 0"/>
+      <origin xyz="${rear_wheel_x} ${reflect*wheel_y} ${wheel_radius}" rpy="0 0 0"/>
       <axis xyz="0 1 0"/>
+      <dynamics damping="0.5" friction="0.8"/>
+      <!-- <limit lower="-3.14159" upper="3.14159" effort="70" velocity="-1"/> -->
     </joint>
     <link name="${prefix}_wheel">
@@ -114,37 +136,41 @@
       </collision>
       <inertial>
-        <mass value="1.0"/>
+        <mass value="${wheel_mass}"/>
         <origin xyz="0 0 0" rpy="0 0 0"/>
-        <inertia ixx="0.005" ixy="0" ixz="0" iyy="0.005" iyz="0" izz="0.005"/>
+        <inertia ixx="${wheel_mass/12*(3*wheel_radius*wheel_radius + wheel_width*wheel_width)}"
+                 ixy="0" ixz="0"
+                 iyy="${wheel_mass/12*(3*wheel_radius*wheel_radius + wheel_width*wheel_width)}"
+                 iyz="0"
+                 izz="${wheel_mass/2 * wheel_radius*wheel_radius}"/>
       </inertial>
     </link>
   </xacro:macro>
   <!-- 实例化轮子 -->
-  <xacro:front_wheel prefix="left_front" reflect="1"/>
-  <xacro:front_wheel prefix="right_front" reflect="-1"/>
-  <xacro:rear_wheel prefix="left_rear" reflect="1"/>
-  <xacro:rear_wheel prefix="right_rear" reflect="-1"/>
+  <xacro:front_wheel prefix="fr_left" reflect="1"/>
+  <xacro:front_wheel prefix="fr_right" reflect="-1"/>
+  <xacro:rear_wheel prefix="re_left" reflect="1"/>
+  <xacro:rear_wheel prefix="re_right" reflect="-1"/>
   <!-- Gazebo材质与摩擦配置 -->
-  <gazebo reference="base_link">
+  <gazebo reference="chassis_link">
     <material>Gazebo/White</material>
     <mu1>0.5</mu1>
     <mu2>0.5</mu2>
   </gazebo>
-  <gazebo reference="left_front_wheel">
+  <gazebo reference="fr_left_wheel">
     <material>Gazebo/Grey</material>
     <mu1>150.0</mu1>
     <mu2>10.0</mu2>
   </gazebo>
-  <gazebo reference="right_front_wheel">
+  <gazebo reference="fr_right_wheel">
     <material>Gazebo/Grey</material>
     <mu1>150.0</mu1>
     <mu2>10.0</mu2>
   </gazebo>
-  <gazebo reference="left_rear_wheel">
+  <gazebo reference="re_left_wheel">
     <material>Gazebo/Grey</material>
     <mu1>150.0</mu1>
     <mu2>10.0</mu2>
   </gazebo>
-  <gazebo reference="right_rear_wheel">
+  <gazebo reference="re_right_wheel">
     <material>Gazebo/Grey</material>
     <mu1>150.0</mu1>
@@ -156,5 +182,5 @@
   <!-- 摄像头：前轮水平位置，宽度一半处 -->
   <joint name="camera_joint" type="fixed">
-    <parent link="base_link"/>
+    <parent link="chassis_link"/>
     <child link="camera_link"/>
     <origin xyz="${front_wheel_x} 0 ${chassis_height}" rpy="0 0 0"/>
@@ -181,5 +207,5 @@
   <!-- 雷达：摄像头往后3cm -->
   <joint name="laser_joint" type="fixed">
-    <parent link="base_link"/>
+    <parent link="chassis_link"/>
     <child link="laser_link"/>
     <origin xyz="${front_wheel_x - 0.03} 0 ${chassis_height}" rpy="0 0 0"/>
@@ -245,5 +271,5 @@
   </gazebo>
   <joint name="imu_joint" type="fixed">
-    <parent link="base_link"/>
+    <parent link="chassis_link"/>
     <child link="imu_link"/>
     <origin xyz="0 0 ${chassis_height/2}" rpy="0 0 0"/>
@@ -360,5 +386,5 @@
   <joint name="virtual_steering_wheel_joint" type="revolute">
     <origin xyz="${-chassis_length/2 + 0.1} 0.0 0.0" rpy="0.0 0.0 0.0"/>
-    <parent link="base_link"/>
+    <parent link="chassis_link"/>
     <child link="virtual_steer_link"/>
     <axis xyz="-1 0 0"/>
@@ -369,10 +395,10 @@
             filename="libgazebo_ros_joint_state_publisher.so">
       <update_rate>100</update_rate>
-      <joint_name>right_front_steer_joint</joint_name>
-      <joint_name>right_front_wheel_joint</joint_name>
-      <joint_name>left_front_steer_joint</joint_name>
-      <joint_name>left_front_wheel_joint</joint_name>
-      <joint_name>right_rear_wheel_joint</joint_name>
-      <joint_name>left_rear_wheel_joint</joint_name>
+      <joint_name>fr_right_steer_joint</joint_name>
+      <joint_name>fr_right_wheel_joint</joint_name>
+      <joint_name>fr_left_steer_joint</joint_name>
+      <joint_name>fr_left_wheel_joint</joint_name>
+      <joint_name>re_right_wheel_joint</joint_name>
+      <joint_name>re_left_wheel_joint</joint_name>
       <joint_name>virtual_steering_wheel_joint</joint_name>
     </plugin>
@@ -395,10 +421,10 @@
       <update_rate>100.0</update_rate>
       <!-- wheels -->
-      <front_left_joint>left_front_wheel_joint</front_left_joint>
-      <front_right_joint>right_front_wheel_joint</front_right_joint>
-      <rear_left_joint>left_rear_wheel_joint</rear_left_joint>
-      <rear_right_joint>right_rear_wheel_joint</rear_right_joint>
-      <left_steering_joint>left_front_steer_joint</left_steering_joint>
-      <right_steering_joint>right_front_steer_joint</right_steering_joint>
+      <front_left_joint>fr_left_wheel_joint</front_left_joint>
+      <front_right_joint>fr_right_wheel_joint</front_right_joint>
+      <rear_left_joint>re_left_wheel_joint</rear_left_joint>
+      <rear_right_joint>re_right_wheel_joint</rear_right_joint>
+      <left_steering_joint>fr_left_steer_joint</left_steering_joint>
+      <right_steering_joint>fr_right_steer_joint</right_steering_joint>
       <steering_wheel_joint>virtual_steering_wheel_joint</steering_wheel_joint>
       <!-- Max absolute steer angle for tyre in radians-->

Commit message: [lucifer][add]: find reason and use real world

File: src/tianbot_description_ros2/urdf/tianbot_ackermann.urdf.xacro (robot description, xacro)
@@ -80,5 +80,5 @@
       <axis xyz="0 1 0"/>
       <dynamics damping="0.5" friction="0.8"/>
-      <!-- <limit lower="-3.14159" upper="3.14159" effort="200" velocity="-1"/> -->
+      <limit lower="-3.14159" upper="3.14159" effort="200" velocity="-1"/>
     </joint>
     <link name="${prefix}_wheel">
@@ -117,5 +117,5 @@
       <axis xyz="0 1 0"/>
       <dynamics damping="0.5" friction="0.8"/>
-      <!-- <limit lower="-3.14159" upper="3.14159" effort="70" velocity="-1"/> -->
+      <limit lower="-3.14159" upper="3.14159" effort="70" velocity="-1"/>
     </joint>
     <link name="${prefix}_wheel">

File: src/tianbot_description_ros2/urdf/tianracer_base.xacro (robot description, xacro)
@@ -42,6 +42,6 @@
                 <box size="${chassis_length} ${chassis_width} ${chassis_height}" />
             </geometry>
-            <material name="gray">
-                <color rgba="0.5 0.5 0.5 1.0" />
+            <material name="black">
+                <color rgba="0.15 0.15 0.15 1.0" />
             </material>
         </visual>

Commit message: [lucifer][add]: try to turn until robot face the  contracy side

File: src/tianbot_description_ros2/urdf/tianbot_ackermann.urdf.xacro (robot description, xacro)
@@ -1,6 +1,6 @@
 <?xml version="1.0"?>
 <robot name="tianbot_ackermann" xmlns:xacro="http://www.ros.org/wiki/xacro">
-  <!-- 实际尺寸参数 -->
-  <xacro:property name="chassis_length" value="0.63"/>
+  <!-- 实际尺寸参数（根据实测调整） -->
+  <xacro:property name="chassis_length" value="0.60"/>
   <xacro:property name="chassis_width" value="0.40"/>
   <xacro:property name="chassis_height" value="0.40"/>
@@ -9,7 +9,8 @@
   <xacro:property name="wheel_mass" value="3.0"/>
   <xacro:property name="steering_mass" value="0.01"/>
-  <!-- 轮子位置：前轮距前端6cm，后轮距后端4cm -->
-  <xacro:property name="front_wheel_x" value="${chassis_length/2 - 0.06}"/>
-  <xacro:property name="rear_wheel_x" value="${-chassis_length/2 + 0.04}"/>
+  <!-- 轮子位置：前轮距前端13cm，后轮距后端7cm（实测值） -->
+  <!-- 轴距 = 0.60 - 0.13 - 0.07 = 0.40m -->
+  <xacro:property name="front_wheel_x" value="${chassis_length/2 - 0.13}"/>
+  <xacro:property name="rear_wheel_x" value="${-chassis_length/2 + 0.07}"/>
   <xacro:property name="wheel_y" value="${chassis_width/2}"/>
   <xacro:property name="wheelbase" value="${front_wheel_x - rear_wheel_x}"/>
